Commit message: works apart from bag files & tactile sensors

File: balancing_grasping/urdf/balancing_grasping.urdf.xacro (robot description, xacro)
@@ -33,7 +33,7 @@
     <visual>
       <geometry>
-	<box size="0.2 0.12 0.01" />
+	<box size="0.1 0.3 0.01" />
       </geometry>
-      <origin rpy="0 0 0" xyz="0 0 0" />
+      <origin rpy="0 0 0" xyz="0 0 0.005" />
     </visual>
   </link>

Commit message: kth robot setup

File: balancing_grasping/urdf/balancing_grasping.urdf.xacro (robot description, xacro)
@@ -9,4 +9,6 @@
   <!--Import the yumi servo gripper macro -->
   <xacro:include filename="$(find yumi_description)/urdf/Grippers/yumi_servo_gripper.xacro"/>
+  <!--Import the yumi optodaq sensors macro -->
+  <xacro:include filename="$(find yumi_description)/urdf/Extras/yumi_optodaq_sensors.xacro"/>
   <!-- Import Gazebo plugins -->
   <xacro:include filename="$(find yumi_description)/urdf/Gazebo/gazebo.urdf.xacro"/>
@@ -15,13 +17,19 @@
     <origin xyz="0 0 0.1" rpy="0 0 0" />
   </xacro:yumi>
-  <!--right gripper-->
-  <xacro:yumi_servo_gripper name="gripper_r" hardware_interface="hardware_interface/$(arg grippers_interface)" parent="yumi_link_7_r">
-    <origin xyz="0 0 0.007" rpy="0 0 ${PI}" />
-  </xacro:yumi_servo_gripper>
-  <!--left gripper-->
-  <xacro:yumi_servo_gripper name="gripper_l" hardware_interface="hardware_interface/$(arg grippers_interface)" parent="yumi_link_7_l">
-    <origin xyz="0 0 0.007" rpy="0 0 ${PI}" />
-  </xacro:yumi_servo_gripper>
-     <xacro:property name="yumi_parent" value="world" />
+ <xacro:yumi_optodaq_sensor name="optodaq_r" parent="yumi_link_7_r">
+     <origin xyz="0 0 0.033" rpy="0 ${PI} -0.7" />
+ </xacro:yumi_optodaq_sensor>
+ <xacro:yumi_optodaq_sensor name="optodaq_l" parent="yumi_link_7_l">
+   <origin xyz="0 0 0.033" rpy="0 ${PI} -0.7" />
+ </xacro:yumi_optodaq_sensor>
+ <!--right gripper-->
+ <xacro:yumi_servo_gripper name="gripper_r" hardware_interface="hardware_interface/EffortJointInterface" parent="optodaq_r_sensor_link">
+   <origin xyz="0 0 -0.033" rpy="0 ${-PI} ${PI}" />
+ </xacro:yumi_servo_gripper>
+ <!--left gripper-->
+ <xacro:yumi_servo_gripper name="gripper_l" hardware_interface="hardware_interface/EffortJointInterface" parent="optodaq_l_sensor_link">
+   <origin xyz="0 0 -0.033" rpy="0 ${-PI} ${PI}" />
+ </xacro:yumi_servo_gripper>
+    <xacro:property name="yumi_parent" value="world" />
     <link name="world"/>
     <joint name="world_joint" type="fixed">
@@ -38,5 +46,5 @@
     </visual>
   </link>
-  <joint name="object_joint" type="floating">
+  <joint name="object_joint" type="fixed">
     <parent link="yumi_base_link" />
     <child link = "obj_frame" />

Commit message: fixed urdf

File: balancing_grasping/urdf/balancing_grasping.urdf.xacro (robot description, xacro)
@@ -25,9 +25,9 @@
  <!--right gripper-->
  <xacro:yumi_servo_gripper name="gripper_r" hardware_interface="hardware_interface/EffortJointInterface" parent="optodaq_r_sensor_link">
-   <origin xyz="0 0 -0.033" rpy="0 ${-PI} ${PI}" />
+   <origin xyz="0 0 -0.033" rpy="${PI} 0.0 ${PI/4}" />
  </xacro:yumi_servo_gripper>
  <!--left gripper-->
  <xacro:yumi_servo_gripper name="gripper_l" hardware_interface="hardware_interface/EffortJointInterface" parent="optodaq_l_sensor_link">
-   <origin xyz="0 0 -0.033" rpy="0 ${-PI} ${PI}" />
+   <origin xyz="0 0 -0.033" rpy="${PI} 0.0 ${PI/4}" />
  </xacro:yumi_servo_gripper>
     <xacro:property name="yumi_parent" value="world" />

Commit message: fixed urdf

File: balancing_grasping/urdf/balancing_grasping.urdf.xacro (robot description, xacro)
@@ -18,8 +18,8 @@
   </xacro:yumi>
  <xacro:yumi_optodaq_sensor name="optodaq_r" parent="yumi_link_7_r">
-     <origin xyz="0 0 0.033" rpy="0 ${PI} -0.7" />
+     <origin xyz="0 0 0.033" rpy="0 ${PI} ${-PI/4}" />
  </xacro:yumi_optodaq_sensor>
  <xacro:yumi_optodaq_sensor name="optodaq_l" parent="yumi_link_7_l">
-   <origin xyz="0 0 0.033" rpy="0 ${PI} -0.7" />
+   <origin xyz="0 0 0.033" rpy="0 ${PI} ${-PI/4}" />
  </xacro:yumi_optodaq_sensor>
  <!--right gripper-->
